File: layout/keyboard.kicad_pcb (KiCad board)
At the start: 2 copper layers, 271.5 x 95.3 mm, 113 parts, among them U1 ProMicro

Commit message: fix gnd
Parts:
- moved D_COMMA1 0.32 mm to (252.4, 109.5)
Connections:
- U1 pad 23: +5V -> GND
- U1 pad 3: Net-(U1-Pad3) -> GND
- U1 pad 4: Net-(U1-Pad4) -> GND
Routing:
- net col3: track 175.6 -> 176.2 mm
- added copper zone on B.Cu, net GND
- added copper zone on F.Cu, net GND
