File: layout/bottom_plate.kicad_pcb (KiCad board)
At the start: 2 copper layers, 293.7 x 117.5 mm, 9 parts

Commit message: Updating with latest stuff
Parts:
- removed the G*** at (67.5, 50.8)
- added G***: LOGO, silkscreens:sb_back_logo, B.Cu at (193.7, 109.5)
- added G***: LOGO, silkscreens:bottom_logo, F.Cu at (54.8, 91.3)
- added REF**: MountingHole_4.3mm_M4, MountingHole:MountingHole_4.3mm_M4, F.Cu at (309.6, 39.7)
- added REF**: MountingHole_4.3mm_M4, MountingHole:MountingHole_4.3mm_M4, F.Cu at (79.4, 39.7)
Other:
- outline, holes or cut-outs redrawn
