File: layout/plate.kicad_pcb (KiCad board)
At the start: 2 copper layers, 293.7 x 117.5 mm, 9 parts

Commit message: Updating with latest stuff
Parts:
- removed the G*** at (67.5, 50.8)
- added G***: LOGO, silkscreens:stars_ss, F.Cu at (196.1, 90.5)
- added G***: LOGO, silkscreens:plate_corner_logo, F.Cu at (315.1, 131.8)
